Commit message: put camera to the front

File: src/ros_project/ros_project_description/urdf/ros_project.main.xacro (robot description, xacro)
@@ -31,5 +31,5 @@
    <joint name="camera_joint" type="fixed">
     <axis xyz="0 0 0" />
-    <origin xyz="0 0 0.1" rpy="0 0 0"/>
+    <origin xyz="0.15 0 0.1" rpy="0 0 0"/>
     <parent link="chassis_main"/>
     <child link="camera_link"/>

File: src/ros_project/ros_project_description/urdf/ros_project.materials.xacro (robot description, xacro)
@@ -10,3 +10,6 @@
     <color rgba="0 1 0 1"/>
   </material>
+  <material name="transparent_black">
+    <color rgba="0 0 0 0.5"/>
+  </material>
 </robot>
