Commit message: changed cylinder to box and made scripts executable

File: src/ros_project/ros_project_description/urdf/ros_project.macros.xacro (robot description, xacro)
@@ -74,5 +74,5 @@
          <visual>
             <geometry>
-               <cylinder length="0.1" radius="${radius}" />
+               <box size="0.4 0.3 0.1"/>
             </geometry>
             <material name="red" />
@@ -80,5 +80,5 @@
          <collision>
             <geometry>
-               <cylinder length="0.1" radius="${radius}" />
+               <box size="0.4 0.3 0.1"/>
             </geometry>
             <origin rpy="0 0 0"/>

Commit message: changed shape of robot and put camera towards the front

File: src/ros_project/ros_project_description/urdf/ros_project.macros.xacro (robot description, xacro)
@@ -74,5 +74,5 @@
          <visual>
             <geometry>
-               <box size="0.4 0.3 0.1"/>
+               <box size="0.3 0.3 0.1"/>
             </geometry>
             <material name="red" />
@@ -80,5 +80,5 @@
          <collision>
             <geometry>
-               <box size="0.4 0.3 0.1"/>
+               <box size="0.3 0.3 0.1"/>
             </geometry>
             <origin rpy="0 0 0"/>
@@ -92,3 +92,25 @@
       </joint>
    </xacro:macro>
+   <xacro:macro name="create_chassis_head" params="radius parent_name xyz">
+      <link name="chassis_head">
+         <visual>
+            <geometry>
+               <box size="0.2 0.2 0.05"/>
+            </geometry>
+            <material name="red" />
+         </visual>
+         <collision>
+            <geometry>
+               <box size="0.2 0.2 0.05"/>
+            </geometry>
+            <origin rpy="0 0 0"/>
+         </collision>
+         <xacro:cylinder_inertia mass="${chassis_mass}" radius="${radius*3}" length="0.1"/>
+      </link>
+      <joint name="chassis_to_chassis_head" type="fixed">
+         <parent link="${parent_name}" />
+         <child link="chassis_head" />
+         <origin xyz="${xyz}" />
+      </joint>
+   </xacro:macro>
 </robot>

File: src/ros_project/ros_project_description/urdf/ros_project.main.xacro (robot description, xacro)
@@ -8,4 +8,5 @@
   <link name="the_world"/>
   <xacro:create_chassis chassis_id = "main" parent_name = "the_world" radius="$(arg chassis_radius)" xyz="0.5 3.2 0.5"/>
+  <xacro:create_chassis_head parent_name = "chassis_main" radius="$(arg chassis_radius)" xyz="0.1 0 0"/>
   <xacro:create_wheel wheel_id = "left" parent_name = "chassis_main" radius="$(arg wheel_radius)" xyz="0 0.15 -0.041"/>
   <xacro:create_wheel wheel_id = "right" parent_name = "chassis_main" radius="$(arg wheel_radius)" xyz="0 -0.15 -0.041"/>
@@ -32,5 +33,5 @@
     <axis xyz="0 0 0" />
     <origin xyz="0 0 0.05" rpy="0 0 0"/>
-    <parent link="chassis_main"/>
+    <parent link="chassis_head"/>
     <child link="camera_link"/>
   </joint>

Commit message: fixed mass and inertia

File: src/ros_project/ros_project_description/urdf/ros_project.macros.xacro (robot description, xacro)
@@ -13,5 +13,17 @@
       </inertial>
    </xacro:macro>
-      <xacro:macro name="sphere_inertia" params="mass radius">
+   <xacro:macro name="box_inertia" params="mass w d h">
+      <inertial>
+         <mass value="${mass}"/>
+         <inertia
+         ixx="${(1/12)*mass*(w**2 + d**2)}"
+         ixy="0.0"
+         ixz="0.0"
+         iyy="${(1/12)*mass*(d**2 + h**2)}"
+         iyz="0.0"
+         izz="${(1/12)*mass*(h**2 + w**2)}" />
+      </inertial>
+   </xacro:macro>
+   <xacro:macro name="sphere_inertia" params="mass radius">
       <inertial>
          <mass value="${mass}"/>
@@ -84,5 +96,5 @@
             <origin rpy="0 0 0"/>
          </collision>
-         <xacro:cylinder_inertia mass="${chassis_mass}" radius="${radius*3}" length="0.1"/>
+      <xacro:box_inertia mass="50" w="0.3" d="0.3" h="0.1"/>
       </link>
       <joint name="world_to_chassis_${chassis_id}" type="fixed">
@@ -106,5 +118,5 @@
             <origin rpy="0 0 0"/>
          </collision>
-         <xacro:cylinder_inertia mass="${chassis_mass}" radius="${radius*3}" length="0.1"/>
+      <xacro:box_inertia mass="10" w="0.2" d="0.2" h="0.05"/>
       </link>
       <joint name="chassis_to_chassis_head" type="fixed">
